File: Power schematics.kicad_sch (KiCad schematic)
At the start: 0 parts

Commit message: Error on the power schematic fixed, recuperated circuit from backup
Parts:
- added C801, C802: 10u 35V, symbol Device:C
- added C803, C804, C808, C810, C811, C813: 0u1, symbol Device:C
- added C805: 10u 16v, symbol Device:C
- added C806, C809, C812, C814: 10u, symbol Device:C
- added C807: 47u 16v, symbol Device:C
- added CR801: B560CQ-13-F, CR_0CQ-13-F_DIO, symbol B560CQ-13-F:B560CQ-13-F
- added D801: LED, symbol Device:LED
- added L801: L, symbol Device:L
- added NR111E801: ~, symbol MyLibrary:NR111D
- added R801: R, symbol Device:R
- added R802: 22, symbol Device:R
- added R803: 2K7, symbol Device:R
- added R804: 1.7M, symbol Device:R
- added R805: 18k, symbol Device:R
- added R806: 3k9, symbol Device:R
- added R807: 0R, symbol Device:R
- added U801, U802: AMS1117-3.3, Package_TO_SOT_SMD:SOT-223-3_TabPin2, symbol Regulator_Linear:AMS1117-3.3
Connections:
- new net: D801.2 (A), R801.2
- new net: NR111E801.7 (EN), R804.2
- new net: C803.2, CR801.1, L801.1, NR111E801.3 (SW)
- new net: NR111E801.1 (BS), R802.2
- new net: NR111E801.5 (FB), R805.1, R806.2
- new net: NR111E801.6 (ISET), R807.2
- new net: C810.1, NR111E801.8 (SS)
- new net: R803.1, R805.2
- new net: C803.1, R802.1
- new net +24V: C801.1, C802.1, NR111E801.2 (IN), R804.1
- new net +3.3V: C813.1, C814.1, U802.2 (VO)
- new net +5V: C804.1, C805.1, C806.1, C807.1, C811.1, C812.1, L801.2, R801.1, R803.2, U801.3 (VI), U802.3 (VI)
- new net GND: C801.2, C802.2, C804.2, C805.2, C806.2, C807.2, C808.2, C809.2, C810.2, C811.2, C812.2, C813.2, C814.2, CR801.2, D801.1 (K), NR111E801.4 (GND), R806.1, R807.1, U801.1 (GND), U802.1 (GND)
- new net VDD: C808.1, C809.1, U801.2 (VO)
